File: MTS_Card_Template.kicad_pcb (KiCad board)
At the start: 6 copper layers, 160 x 100 mm, 14 parts, among them J1 DIN41612_02x16_ZB, SW1 SW_DIP_x04, U1 TCAN337GDR, U3 24LC32, U4 LM75B

Commit message: Edit Connector
Parts:
- removed C1: 100n, Capacitor_SMD:C_0805_2012Metric_Pad1.18x1.45mm_HandSolder
- removed U4: LM75B, Package_SO:MSOP-8_3x3mm_P0.65mm
- moved QR Code 64.2 mm to (154.5, 113.0)
- moved QR Code 64.0 mm to (154.5, 113.0)
- moved C3 33.8 mm to (214.0, 82.9), turned to 90 degrees
- moved U3 12.2 mm to (219.5, 98.1)
- moved D2 2.27 mm to (230.5, 83.1)
- moved D3 2.27 mm to (230.5, 88.2)
- moved U1 2.27 mm to (221.5, 83.1)
- moved J1 1.48 mm to (238.8, 81.8)
Routing:
- net +3V3: track 5.86 -> 12.5 mm, vias 1 -> 2
- net GND: track 9.64 -> 11.0 mm, vias 3 -> 4
- net a4: track 0.00 -> 0.96 mm
- net a3: track 0.96 -> 0.00 mm
- net I2C_BUS_SDA: track 7.35 -> 6.83 mm
Other:
- board text added: "HW Rev.X.X"
- board text added: "Styria Electronics"
- board text removed: "Andras Nagy 2024"
- board text removed: "HW Rev.2.0"

Commit message: Update Connector
Parts:
- removed the QR Code at (154.5, 113.0)
- removed SW1: SW_DIP_x04, Button_Switch_SMD:SW_DIP_SPSTx04_Slide_6.7x11.72mm_W8.61mm_P2.54mm_LowProfile
- removed U3: 24LC32, Package_SO:SOIC-8_3.9x4.9mm_P1.27mm
- added C1: 100nF, Capacitor_SMD:C_0805_2012Metric_Pad1.18x1.45mm_HandSolder, F.Cu at (160.8, 79.3)
- added C4: 100nF, Capacitor_SMD:C_0805_2012Metric_Pad1.18x1.45mm_HandSolder, F.Cu at (160.8, 82.3)
- added C5: 47µF, Capacitor_SMD:C_1210_3225Metric, F.Cu at (136.6, 88.4)
- added C6: 47µF, Capacitor_SMD:C_1210_3225Metric, F.Cu at (136.6, 92.7)
- added D1: PESD3V3L2BT, Package_TO_SOT_SMD:SOT-23, F.Cu at (141.9, 80.2)
- added F1: Fuse, Fuse:Fuse_1206_3216Metric, F.Cu at (147.1, 79.5)
- added F2: Fuse, Fuse:Fuse_1206_3216Metric, F.Cu at (147.1, 82.8)
- added R1: 0.20Ω, Resistor_SMD:R_1206_3216Metric, F.Cu at (147.1, 86.1)
- added R2: 0.20Ω, Resistor_SMD:R_1206_3216Metric, F.Cu at (147.1, 89.4)
- added U2: INA219AxD, Package_SO:SOIC-8_3.9x4.9mm_P1.27mm, F.Cu at (154.2, 87.7)
- C2, C3: value 100n -> 47µF; footprint Capacitor_SMD:C_0805_2012Metric_Pad1.18x1.45mm_HandSolder -> Capacitor_SMD:C_1210_3225Metric
- U1: value TCAN337GDR -> INA219AxD
- moved QR Code 137.8 mm to (20.5, 80.5)
- moved C2 92.1 mm to (136.6, 79.9), turned to 0 degrees
- moved D3 88.6 mm to (141.9, 89.5)
- moved D2 88.6 mm to (141.9, 84.8)
- moved C3 77.4 mm to (136.6, 84.2), turned to 0 degrees
- moved U1 67.4 mm to (154.2, 81.2)
- moved J1 1.44 mm to (238.9, 83.2)
Connections:
- net a3 renamed /Conn/SLOT_ID
- net a5 renamed /Conn/TXB-
- net a6 renamed /Conn/TXB+
- net a7 renamed /Conn/RXB-
- net a8 renamed /Conn/RXB+
- net b10 renamed UBAT
- net b5 renamed /Conn/TXA+
- net b6 renamed /Conn/TXA-
- net b7 renamed /Conn/RXA+
- net b8 renamed /Conn/RXA-
- C2 pad 1: +3V3 -> +3V3Ext
- C3 pad 1: +3V3 -> +3V3Ext
- D2 pad 1: /CANH -> /Conn/I2C_BUS_CLK
- D2 pad 2: /CANL -> /Conn/I2C_BUS_SDA
- D3 pad 1: I2C_BUS_SDA -> /Conn/CAN_L
- D3 pad 2: I2C_BUS_CLK -> /Conn/CAN_H
- J1 pad a1: /Triger -> /Conn/Triger
- J1 pad a2: a2 -> /Conn/SYNC_CPU
- J1 pad b1: /CANH -> /Conn/CAN_H
- J1 pad b2: /CANL -> /Conn/CAN_L
- J1 pad b3: I2C_BUS_SDA -> /Conn/I2C_BUS_SDA
- J1 pad b4: I2C_BUS_CLK -> /Conn/I2C_BUS_CLK
- U1 pad 1: CANFD_TX -> GND
- U1 pad 3: +3V3 -> I2C1_SDA
- U1 pad 4: CANFD_RX -> I2C1_SCL
- U1 pad 5: unconnected-(U1-VIO-Pad5) -> +3V3
- U1 pad 6: /CANL -> GND
- U1 pad 7: /CANH -> +3V3
- U1 pad 8: unconnected-(U1-STB-Pad8) -> Net-(U1-IN+)
Routing:
- net /CANH: track 13.2 -> 0.00 mm
- net /CANL: track 13.1 -> 0.00 mm
- net +3V3: track 12.5 -> 0.00 mm, vias 2 -> 0
- net GND: track 11.0 -> 0.00 mm, vias 4 -> 0
- net I2C_BUS_SDA: track 6.83 -> 0.00 mm
- net I2C_BUS_CLK: track 6.75 -> 0.00 mm
- net +3V3Ext: track 2.62 -> 0.00 mm
- net CANFD_RX: track 2.56 -> 0.00 mm, vias 1 -> 0
- net +5VExt: track 2.54 -> 0.00 mm
- net CANFD_TX: track 2.50 -> 0.00 mm, vias 1 -> 0
- net a4: track 0.96 -> 0.00 mm
- net /Conn/SLOT_ID: track 0.00 -> 0.96 mm
