File: MTS_Card_Template.kicad_sch (KiCad schematic)
At the start: 10 parts, among them J1 DIN41612_02x16_ZB, SW1 SW_DIP_x04, U1 TCAN337GDR, U3 24LC32, U4 LM75B

Commit message: Edit Connector
Parts:
- removed C1: 100n, Capacitor_SMD:C_0805_2012Metric_Pad1.18x1.45mm_HandSolder, symbol Device:C_Small
- removed U4: LM75B, Package_SO:MSOP-8_3x3mm_P0.65mm, symbol Sensor_Temperature:LM75B

Commit message: Update Connector
Parts:
- removed C2, C3: 100n, Capacitor_SMD:C_0805_2012Metric_Pad1.18x1.45mm_HandSolder, symbol Device:C_Small
- removed D2, D3: PESD2CANFD24V-T, Package_TO_SOT_SMD:SOT-23, symbol Power_Protection:SP0502BAHT
- removed J1: DIN41612_02x16_ZB, Connector_DIN:DIN41612_B2_2x16_Male_Horizontal_THT, symbol Connector:DIN41612_02x16_ZB
- removed SW1: SW_DIP_x04, Button_Switch_SMD:SW_DIP_SPSTx04_Slide_6.7x11.72mm_W8.61mm_P2.54mm_LowProfile, symbol Switch:SW_DIP_x04
- removed U1: TCAN337GDR, Package_SO:SOIC-8_3.9x4.9mm_P1.27mm, symbol Interface_CAN_LIN:TJA1042T-3
- removed U3: 24LC32, Package_SO:SOIC-8_3.9x4.9mm_P1.27mm, symbol Memory_EEPROM:24LC32
Other:
- added sheet Conn (Conn.kicad_sch)
- note removed: "I2C Address 0xA0"
- note removed: "place near as possible to connector"
